File: docs/Schematics/pico-106.kicad_pcb (KiCad board)
At the start: 2 copper layers, 13 x 1.4 mm, 31 parts, among them J2 Debug, J3 Stereo line out, J4 Debug, SW1 RST, U1 MCU arm Cortex-M0x2, U2 I2S DAC, U3 H11L1, U4 74HCT374, U5 74HCT374, U6 D1X8K-14BL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

Commit message: Capture latest docs
Parts:
- removed DS1: HY1602E, Display:HY1602E
- removed R10, R11, R12, R13, R14, R15, R16, R17, R18: 330, Resistor_THT:R_Axial_DIN0204_L3.6mm_D1.6mm_P5.08mm_Horizontal
- removed U4, U5: 74HCT374, Package_DIP:DIP-20_W7.62mm_LongPads
- removed U6, U7: D1X8K-14BL, Display_7Segment:D1X8K
- added C1: 22nF, Capacitor_THT:C_Disc_D5.0mm_W2.5mm_P5.00mm, F.Cu at (127.0, 71.1)
- added C2: 220pF, Capacitor_THT:C_Disc_D5.0mm_W2.5mm_P5.00mm, F.Cu at (116.8, 83.8)
- added C3: 1nF, Capacitor_THT:C_Disc_D5.0mm_W2.5mm_P5.00mm, F.Cu at (78.8, 127.0)
- added C4: 22nF, Capacitor_THT:C_Disc_D5.0mm_W2.5mm_P5.00mm, F.Cu at (43.2, 137.2)
- added Q1: 2N2222A, Package_TO_SOT_THT:TO-92, F.Cu at (66.0, 81.3)
- R2: value 1K -> 33k
- R3: value 330 -> 27k
- R4, R9: value 330 -> 33k
- R5: value 330 -> 220k
- R6: value 330 -> 1.8k
- R7: value 330 -> 47k
- R8: value 330 -> 2.2k
- U1: value MCU arm Cortex-M0x2 -> Pico 2 (RP2350); footprint Package_DIP:DIP-40_W25.4mm_Socket_LongPads -> Package_DIP:DIP-40_W25.4mm_Socket
- U2: value I2S DAC -> TL072; footprint Package_DIP:DIP-40_W25.4mm_Socket_LongPads -> Package_DIP:DIP-8_W7.62mm_Socket
- moved J3 228.2 mm to (38.2, 172.6)
- moved U2 150.3 mm to (83.8, 111.8), turned to 90 degrees
- moved R9 133.4 mm to (43.2, 149.8), turned to -90 degrees
- moved SW1 133.3 mm to (184.7, 46.0)
- moved R8 115.2 mm to (61.0, 142.2), turned to 90 degrees
- moved U1 111.9 mm to (162.6, 76.2)
- moved J4 101.3 mm to (162.6, 35.6)
- moved R5 99.1 mm to (73.7, 101.6), turned to -90 degrees
- moved R6 95.2 mm to (88.9, 83.8), turned to 180 degrees
- moved R4 88.0 mm to (88.9, 91.4), turned to 180 degrees
- moved R7 83.0 mm to (101.6, 83.8), turned to 90 degrees
- moved U3 67.6 mm to (208.3, 96.5)
- moved J2 65.7 mm to (147.3, 76.2), turned to -90 degrees
- moved R3 56.5 mm to (127.0, 88.9), turned to 180 degrees
- moved R2 45.8 mm to (139.7, 88.9), turned to 180 degrees
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Connections:
- net /MIDI in (RX) 115200 baud 8-N-1 renamed /console RX
- net /console (TX) 115200 baud 8-N-1 renamed /console TX 115200 baud 8-N-1 
- net Net-(J2-Pin_3) renamed /console GND
- J3 pad S: Net-(U2-AUDIO_L) -> unconnected-(J3-PadS)
- J3 pad T: Net-(U2-AUDIO_R) -> Net-(J3-PadT)
- R2 pad 1: Net-(DS1-LEDA) -> Net-(U1-GPIO3)
- R2 pad 2: +5V -> Net-(C1-Pad2)
- R3 pad 1: Net-(U6-A) -> Net-(C1-Pad2)
- R3 pad 2: Net-(U4-Q5) -> Net-(U2B--)
- R4 pad 1: Net-(U6-B) -> Net-(U2B--)
- R4 pad 2: Net-(U4-Q4) -> Net-(R4-Pad2)
- R5 pad 1: Net-(U6-C) -> Net-(R4-Pad2)
- R5 pad 2: Net-(U4-Q2) -> Net-(Q1-E)
- R6 pad 1: Net-(U6-D) -> Net-(C2-Pad2)
- R7 pad 1: Net-(U6-E) -> Net-(C2-Pad2)
- R7 pad 2: Net-(U4-Q0) -> Earth
- R8 pad 2: Net-(U4-Q6) -> Net-(C3-Pad2)
- R9 pad 2: Net-(U4-Q7) -> Net-(J3-PadT)
- U1 pad 10: /D1 -> unconnected-(U1-GPIO7-Pad10)
- U1 pad 11: /D2 -> unconnected-(U1-GPIO8-Pad11)
- U1 pad 12: /D3 -> unconnected-(U1-GPIO9-Pad12)
- U1 pad 14: /D4 -> unconnected-(U1-GPIO10-Pad14)
- U1 pad 15: /D5 -> unconnected-(U1-GPIO11-Pad15)
- U1 pad 16: /D6 -> unconnected-(U1-GPIO12-Pad16)
- U1 pad 17: /D7 -> unconnected-(U1-GPIO13-Pad17)
- U1 pad 19: Net-(DS1-RS) -> unconnected-(U1-GPIO14-Pad19)
- U1 pad 20: Net-(DS1-E) -> unconnected-(U1-GPIO15-Pad20)
- U1 pad 27: unconnected-(U1-GPIO21-Pad27) -> /MIDI 31250 baud 8-N-1
- U1 pad 29: /I2S SD -> unconnected-(U1-GPIO22-Pad29)
- U1 pad 31: /12.568576 MHz -> unconnected-(U1-GPIO26_ADC0-Pad31)
- U1 pad 32: /49.096 KHz -> unconnected-(U1-GPIO27_ADC1-Pad32)
- U1 pad 34: /1.571072 MHz -> unconnected-(U1-GPIO28_ADC2-Pad34)
- U1 pad 38: Earth -> unconnected-(U1-GND-Pad38)
- U1 pad 39: Net-(U1-VSYS) -> +5V
- U1 pad 7: /31250 baud 8-N-1 -> unconnected-(U1-GPIO5-Pad7)
- U1 pad 9: /D0 -> unconnected-(U1-GPIO6-Pad9)
- U2 pad 1: (no net) -> Net-(C3-Pad2)
- U2 pad 2: (no net) -> Net-(Q1-E)
- U2 pad 4: (no net) -> -12V
- U2 pad 5: (no net) -> Earth
- U2 pad 6: (no net) -> Net-(U2B--)
- U2 pad 7: (no net) -> Net-(R4-Pad2)
- U2 pad 8: Earth -> +12V
- U3 pad 4: /31250 baud 8-N-1 -> /MIDI 31250 baud 8-N-1
